File: KiCad Files/M4 Breadstick/LEDs.sch (KiCad schematic (older format))
At the start: 0 parts

Commit message: LEDs moved to child sheet
Parts:
- added RGB1, RGB10, RGB11, RGB12, RGB13, RGB14, RGB15, RGB16, RGB17, RGB18, RGB19, RGB2, RGB20, RGB21, RGB22, RGB23, RGB24, RGB3, RGB33, RGB4, RGB5, RGB6, RGB7, RGB8, RGB9: LC8822-2020, MichaelRangen_Footprints:LC8822-2020, symbol M4-Breadstick-rescue:LC8822-2020-MichaelRangen_SchematicSymbols
- added U1: SN74LVC2T45DCUR, Housings_SSOP:VSSOP-8_2.3x2mm_Pitch0.5mm, symbol Logic_LevelTranslator:74LVC2T45DC
Connections:
- new net: RGB8.2 (CO), RGB9.5 (CI)
- new net: RGB8.3 (DO), RGB9.6 (DI)
- new net: RGB7.2 (CO), RGB8.5 (CI)
- new net: RGB7.3 (DO), RGB8.6 (DI)
- new net: RGB6.2 (CO), RGB7.5 (CI)
- new net: RGB6.3 (DO), RGB7.6 (DI)
- new net: RGB5.2 (CO), RGB6.5 (CI)
- new net: RGB5.3 (DO), RGB6.6 (DI)
- new net: RGB4.2 (CO), RGB5.5 (CI)
- new net: RGB4.3 (DO), RGB5.6 (DI)
- new net: RGB3.2 (CO), RGB4.5 (CI)
- new net: RGB3.3 (DO), RGB4.6 (DI)
- new net: RGB2.2 (CO), RGB3.5 (CI)
- new net: RGB2.3 (DO), RGB3.6 (DI)
- new net: RGB1.2 (CO), RGB2.5 (CI)
- new net: RGB1.3 (DO), RGB2.6 (DI)
- new net: RGB1.5 (CI), U1.2 (1A)
- new net: RGB1.6 (DI), U1.3 (2A)
- new net: RGB23.2 (CO), RGB24.5 (CI)
- new net: RGB23.3 (DO), RGB24.6 (DI)
- new net: RGB22.2 (CO), RGB23.5 (CI)
- new net: RGB22.3 (DO), RGB23.6 (DI)
- new net: RGB21.2 (CO), RGB22.5 (CI)
- new net: RGB21.3 (DO), RGB22.6 (DI)
- new net: RGB20.2 (CO), RGB21.5 (CI)
- new net: RGB20.3 (DO), RGB21.6 (DI)
- new net: RGB19.2 (CO), RGB20.5 (CI)
- new net: RGB19.3 (DO), RGB20.6 (DI)
- new net: RGB18.2 (CO), RGB19.5 (CI)
- new net: RGB18.3 (DO), RGB19.6 (DI)
- new net: RGB17.2 (CO), RGB18.5 (CI)
- new net: RGB17.3 (DO), RGB18.6 (DI)
- new net: RGB16.2 (CO), RGB17.5 (CI)
- new net: RGB16.3 (DO), RGB17.6 (DI)
- new net: RGB15.2 (CO), RGB16.5 (CI)
- new net: RGB15.3 (DO), RGB16.6 (DI)
- new net: RGB14.2 (CO), RGB15.5 (CI)
- new net: RGB14.3 (DO), RGB15.6 (DI)
- new net: RGB13.2 (CO), RGB14.5 (CI)
- new net: RGB13.3 (DO), RGB14.6 (DI)
- new net: RGB12.2 (CO), RGB13.5 (CI)
- new net: RGB12.3 (DO), RGB13.6 (DI)
- new net: RGB11.2 (CO), RGB12.5 (CI)
- new net: RGB11.3 (DO), RGB12.6 (DI)
- new net: RGB10.2 (CO), RGB11.5 (CI)
- new net: RGB10.3 (DO), RGB11.6 (DI)
- new net: RGB10.5 (CI), RGB9.2 (CO)
- new net: RGB10.6 (DI), RGB9.3 (DO)
- new net: U1.4 (GND), U1.5 (DIR)
- new net 5V: RGB1.1 (VDD), RGB10.1 (VDD), RGB11.1 (VDD), RGB12.1 (VDD), RGB13.1 (VDD), RGB14.1 (VDD), RGB15.1 (VDD), RGB16.1 (VDD), RGB17.1 (VDD), RGB18.1 (VDD), RGB19.1 (VDD), RGB2.1 (VDD), RGB20.1 (VDD), RGB21.1 (VDD), RGB22.1 (VDD), RGB23.1 (VDD), RGB24.1 (VDD), RGB3.1 (VDD), RGB4.1 (VDD), RGB5.1 (VDD), RGB6.1 (VDD), RGB7.1 (VDD), RGB8.1 (VDD), RGB9.1 (VDD), U1.1 (VCCA)
- new net LED_STRIP_CLK: U1.7 (1B)
- new net LED_STRIP_DATA: U1.6 (2B)
- new net STATUS_LED_CLK: RGB33.5 (CI)
- new net STATUS_LED_DATA: RGB33.6 (DI)
