File: KiCad Files/M4 Breadstick/Power.sch (KiCad schematic (older format))
At the start: 0 parts

Commit message: page template done
needs review from mike
Parts:
- added C1, C10, C8, C9: CERAMIC-100UF-6.3V-20%-X5R_1206_, OPL_Capacitor:C1206, symbol M4-Breadstick-rescue:CERAMIC-100UF-6.3V-20%-X5R_1206_-OPL_Capacitor
- added C2: 10uF_6.3V_0402_302010053, OPL_Capacitor:C0402, symbol Device:C
- added C3, C4: 1uF_6.3V_0402_302010003, OPL_Capacitor:C0402, symbol Device:C
- added D1, D2: SS24FL, OPL_Discrete_Semiconductor:SOD-123, symbol M4-Breadstick-rescue:SMD-DIODE-SCHOTTKY-20V-1A_SOD-123_-OPL_Discrete_Semiconduc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
- added J21: VBUS, Pin_Headers:Pin_Header_Straight_1x01_Pitch2.54mm, symbol Connector:Conn_01x01_Male
- added J27: VBAT, Pin_Headers:Pin_Header_Straight_1x01_Pitch2.54mm, symbol Connector:Conn_01x01_Male
- added J29, J30: 3.3V, Pin_Headers:Pin_Header_Straight_1x01_Pitch2.54mm, symbol Connector:Conn_01x01_Male
- added U3: NCP1117ST33T3G, digikey-footprints:SOT-223, symbol M4-Breadstick-rescue:NCP1117ST33T3G-MichaelRangen_SchematicSymbols
Connections:
- new net: C2.1, C3.1, C4.1, C8.1, J29.1 (Pin_1), J30.1 (Pin_1), U3.2 (OUT)
- new net: D1.1 (+), J21.1 (Pin_1)
- new net: D2.1 (+), J27.1 (Pin_1)
- new net 5V: C1.1, C10.1, C9.1, D1.2 (-), D2.2 (-), U3.3 (IN)
